File: senseBeRx_rev1/senseBeRx_rev1.sch (KiCad schematic (older format))
At the start: 35 parts, among them J1 Audio-Jack-4_1Switches, J2 Audio-Jack-4_1Switches, P1 CONN_02X05, Q1 SI2301, Q2 Q_NMOS_DGS, Q3 Q_NMOS_DGS, Q4 Q_NMOS_DGS, SW1 SW_DPST, U1 MDBT42Q, U2 TSSP4056, Y1 Crystal

Commit message: Update the part numbers of the components
Parts:
- J1, J2: value Audio-Jack-4_1Switches -> SJ2-35863B1-SMT
- Q2, Q3, Q4: value Q_NMOS_DGS -> SI2302
- Y1: value Crystal -> T38 Mercury
Changed lines of the file:
@@
 P 10425 2275
 F 0 "Q4" H 10575 2150 50  0000 L CNN
-F 1 "Q_NMOS_DGS" H 9900 2400 50  0000 L CNN
+F 1 "SI2302" H 10150 2400 50  0000 L CNN
 F 2 "Package_TO_SOT_SMD:SOT-23_Handsoldering" H 10625 2375 50  0001 C CNN
 F 3 "~" H 10425 2275 50  0001 C CNN
@@
 P 5900 1750
 F 0 "Q3" H 5800 1600 50  0000 L CNN
-F 1 "Q_NMOS_DGS" H 5400 1525 50  0000 L CNN
+F 1 "SI2302" H 5650 1900 50  0000 L CNN
 F 2 "Package_TO_SOT_SMD:SOT-23_Handsoldering" H 6100 1850 50  0001 C CNN
 F 3 "~" H 5900 1750 50  0001 C CNN
@@
 P 5475 1750
 F 0 "Q2" H 5400 1600 50  0000 L CNN
-F 1 "Q_NMOS_DGS" H 5000 1500 50  0000 L CNN
+F 1 "SI2302" H 5275 1900 50  0000 L CNN
 F 2 "Package_TO_SOT_SMD:SOT-23_Handsoldering" H 5675 1850 50  0001 C CNN
 F 3 "~" H 5475 1750 50  0001 C CNN
@@
 P 3750 6550
 F 0 "Y1" H 3750 6700 50  0000 C CNN
-F 1 "Crystal" H 3750 6400 50  0000 C CNN
+F 1 "T38 Mercury" H 3750 6400 50  0000 C CNN
 F 2 "Crystal:Crystal_C38-LF_D3.0mm_L8.0mm_Horizontal" H 3750 6550 50  0001 C CNN
 F 3 "" H 3750 6550 50  0000 C CNN
@@
 P 8850 3850
 F 0 "J1" H 8840 4275 50  0000 C CNN
-F 1 "Audio-Jack-4_1Switches" H 8840 4184 50  0000 C CNN
+F 1 "SJ2-35863B1-SMT" H 8840 4184 50  0000 C CNN
 F 2 "Connector_Audio:Jack_3.5mm_PJ320E_Horizontal" H 9100 3950 50  0001 C CNN
 F 3 "" H 9100 3950 50  0001 C CNN
@@
 P 8875 5600
 F 0 "J2" H 8865 6025 50  0000 C CNN
-F 1 "Audio-Jack-4_1Switches" H 8865 5934 50  0000 C CNN
+F 1 "SJ2-35863B1-SMT" H 8865 5934 50  0000 C CNN
 F 2 "Connector_Audio:Jack_3.5mm_PJ320E_Horizontal" H 9125 5700 50  0001 C CNN
 F 3 "" H 9125 5700 50  0001 C CNN
