File: senseBeTx_rev1/senseBeTx_rev1.sch (KiCad schematic (older format))
At the start: 36 parts, among them J1 Audio-Jack-4_1Switches, P1 CONN_02X05, Q1 TSM2301, Q2 Q_NMOS_DGS, Q3 Q_NMOS_DGS, Q4 Q_NMOS_DGS, Q5 Q_NMOS_DGS, Q6 Q_NMOS_DGS, Q7 Q_NMOS_DGS, Q8 Q_NMOS_DGS, SW1 SW_Push_Dual, U1 STM32L011F3Px, Y1 Crystal

Commit message: Adds notes and proper labeling of Schematic smybols, and PCB Placement of components completed.
Parts:
- added C5: 100nF, Capacitor_SMD:C_0603_1608Metric_Pad1.05x0.95mm_HandSolder, symbol senseBeRx_rev1:C
- D2: value LED_Dual_ACAC -> APBD3224SURKCGKC-F01
- Q1: symbol senseBeRx_rev1:Q_PMOS_DGS -> Device:Q_NMOS_GSD
- Q2, Q3, Q4, Q5, Q6, Q7, Q8: symbol senseBeRx_rev1:Q_NMOS_DGS -> Device:Q_NMOS_GSD
- R10, R6, R7, R8, R9: value 10k -> 100k
- SW1: footprint Button_Switch_THT:SW_PUSH_6mm -> Button_Switch_THT:SW_TH_Tactile_Omron_B3F-10xx
Connections:
- net labels added: 4R7, R12, R20, R_CNTRL
Other:
- note added: "A momentary Push button\n w/ debouncing Cap to \nswitch to config, mode."
- note added: "Ambient Light Sensing"
- note added: "For Programming/Debugging \nthe STM Controller"
- note added: "Infra Red LED Tx"
- note added: "Low Freq. \nCrystal\n32.768 kHz"
- note added: "N-Channel MOSFET Array \nto change Current flowing \nthrough the IR Tx LED."
- note added: "N-Channel MOSFET Array \nto give the IR LED Tx\na pulse input."
- note added: "Port for UART comm. b/w \nSenseBe Rx and Tx units"
- note added: "Reverse Polarity Protection"
- note added: "Two color (Red/Green) LED"
- moved on the sheet: D3

Commit message: Adds schematic files with minor changes, completed PCB files, and Gerber files for manufacturing
Parts:
- Q1: value TSM2301 -> SI2301
- Q2, Q3, Q4, Q5, Q6, Q7, Q8: value Q_NMOS_DGS -> SI2302

Commit message: LED in the design is changed to part no. KPTBD-3216SURKCGKC, updated in schematic and PCB
Parts:
- D2: value APBD3224SURKCGKC-F01 -> KPTBD-3216SURKCGKC; footprint senseBeTx_rev1_fp:LED_APBD3224SURKCGKC-F01 -> senseBeTx_rev1_fp:LED_KPTBD-3216SURKCGKC
Changed lines of the file:
@@
 P 4400 1125
 F 0 "D2" H 4400 1375 50  0000 C CNN
-F 1 "APBD3224SURKCGKC-F01" H 4400 850 50  0000 C CNN
-F 2 "senseBeTx_rev1_fp:LED_APBD3224SURKCGKC-F01" H 4430 1125 50  0001 C CNN
+F 1 "KPTBD-3216SURKCGKC" H 4400 850 50  0000 C CNN
+F 2 "senseBeTx_rev1_fp:LED_KPTBD-3216SURKCGKC" H 4430 1125 50  0001 C CNN
 F 3 "~" H 4430 1125 50  0001 C CNN
 	1    4400 1125
