File: Ap3403_LED_test/Ap3403_LED_test.sch (KiCad schematic (older format))
At the start: 21 parts, among them J1 Batt conn, J2 Conn_01x02, J3 Conn_01x04, Q1 SI2302, Q2 SI2302, Q3 SI2302, U1 AP3403

Commit message: PCB Files completed, ready to manufacture.
Parts:
- C1, C3: footprint (none) -> Ap3403_LED_test_fp:C_0805_HandSoldering; symbol AP3403_LED_test:C -> Ap3403_LED_test-rescue:C-AP3403_LED_test
- C2: footprint (none) -> Ap3403_LED_test_fp:C_0603_HandSoldering; symbol AP3403_LED_test:C -> Ap3403_LED_test-rescue:C-AP3403_LED_test
- D1: footprint (none) -> LED_THT:LED_D5.0mm; symbol AP3403_LED_test:LED -> Ap3403_LED_test-rescue:LED-AP3403_LED_test
- J1: footprint (none) -> Ap3403_LED_test_fp:Molex_KK-6410-02_02x2.54mm_Straight; symbol AP3403_LED_test:Conn_01x02 -> Ap3403_LED_test-rescue:Conn_01x02-AP3403_LED_test
- J2: footprint (none) -> Connector_PinHeader_2.54mm:PinHeader_1x02_P2.54mm_Vertical; symbol AP3403_LED_test:Conn_01x02 -> Ap3403_LED_test-rescue:Conn_01x02-AP3403_LED_test
- J3: footprint (none) -> Connector_PinHeader_2.54mm:PinHeader_1x04_P2.54mm_Vertical; symbol AP3403_LED_test:Conn_01x04 -> Ap3403_LED_test-rescue:Conn_01x04-AP3403_LED_test
- L1: footprint (none) -> Inductor_SMD:L_0805_2012Metric_Pad1.15x1.40mm_HandSolder; symbol AP3403_LED_test:L -> Ap3403_LED_test-rescue:L-AP3403_LED_test
- Q1, Q2, Q3: footprint (none) -> Package_TO_SOT_SMD:SOT-23_Handsoldering; symbol AP3403_LED_test:Q_NMOS_GSD -> Ap3403_LED_test-rescue:Q_NMOS_GSD-AP3403_LED_test
- R1, R2, R3, R4, R5, R6, R7, R8: footprint (none) -> Ap3403_LED_test_fp:R_0603_HandSoldering; symbol AP3403_LED_test:R -> Ap3403_LED_test-rescue:R-AP3403_LED_test
- TP1: footprint (none) -> Ap3403_LED_test_fp:Measurement_Point_Round-SMD-Pad_Small; symbol AP3403_LED_test:Test_Point -> Ap3403_LED_test-rescue:Test_Point-AP3403_LED_test
- U1: footprint (none) -> Ap3403_LED_test_fp:AP3403_U-DFN1616-6(Type G); symbol AP3403_LED_test:AP3403 -> Ap3403_LED_test-rescue:AP3403-AP3403_LED_test
Changed lines of the file:
@@
 $EndDescr
 $Comp
-L AP3403_LED_test:AP3403 U1
+L Ap3403_LED_test-rescue:AP3403-AP3403_LED_test U1
 U 1 1 5C28BCDE
 P 5525 3675
 F 0 "U1" H 5525 4150 50  0000 C CNN
 F 1 "AP3403" H 5525 4059 50  0000 C CNN
-F 2 "" H 5525 3525 50  0001 C CNN
+F 2 "Ap3403_LED_test_fp:AP3403_U-DFN1616-6(Type G)" H 5525 3525 50  0001 C CNN
 F 3 "" H 5525 3525 50  0001 C CNN
 	1    5525 3675
@@
 $EndComp
 $Comp
-L AP3403_LED_test:R R2
+L Ap3403_LED_test-rescue:R-AP3403_LED_test R2
 U 1 1 5C28F0DC
 P 6925 3600
 F 0 "R2" H 6995 3646 50  0000 L CNN
 F 1 "470k" H 6995 3555 50  0000 L CNN
-F 2 "" V 6855 3600 50  0001 C CNN
+F 2 "Ap3403_LED_test_fp:R_0603_HandSoldering" V 6855 3600 50  0001 C CNN
 F 3 "~" H 6925 3600 50  0001 C CNN
 	1    6925 3600
@@
 $EndComp
 $Comp
-L AP3403_LED_test:C C1
+L Ap3403_LED_test-rescue:C-AP3403_LED_test C1
 U 1 1 5C28F1F7
 P 4475 3675
 F 0 "C1" H 4590 3721 50  0000 L CNN
 F 1 "22u" H 4590 3630 50  0000 L CNN
-F 2 "" H 4513 3525 50  0001 C CNN
+F 2 "Ap3403_LED_test_fp:C_0805_HandSoldering" H 4513 3525 50  0001 C CNN
 F 3 "~" H 4475 3675 50  0001 C CNN
 	1    4475 3675
@@
 $EndComp
 $Comp
-L AP3403_LED_test:GND #PWR05
+L Ap3403_LED_test-rescue:GND-AP3403_LED_test #PWR05
 U 1 1 5C28F2CF
 P 6175 4000
@@
 $EndComp
 $Comp
-L AP3403_LED_test:Q_NMOS_GSD Q1
+L Ap3403_LED_test-rescue:Q_NMOS_GSD-AP3403_LED_test Q1
 U 1 1 5C28F427
 P 7575 4575
 F 0 "Q1" H 7475 4425 50  0000 L CNN
 F 1 "SI2302" H 7300 4700 50  0000 L CNN
-F 2 "" H 7775 4675 50  0001 C CNN
+F 2 "Package_TO_SOT_SMD:SOT-23_Handsoldering" H 7775 4675 50  0001 C CNN
 F 3 "~" H 7575 4575 50  0001 C CNN
 	1    7575 4575
@@
 $EndComp
 $Comp
-L AP3403_LED_test:LED D1
+L Ap3403_LED_test-rescue:LED-AP3403_LED_test D1
 U 1 1 5C299534
 P 9725 3750
 F 0 "D1" V 9763 3633 50  0000 R CNN
 F 1 "LED" V 9672 3633 50  0000 R CNN
-F 2 "" H 9725 3750 50  0001 C CNN
+F 2 "LED_THT:LED_D5.0mm" H 9725 3750 50  0001 C CNN
 F 3 "~" H 9725 3750 50  0001 C CNN
 	1    9725 3750
@@
 $EndComp
 $Comp
-L AP3403_LED_test:Conn_01x04 J3
+L Ap3403_LED_test-rescue:Conn_01x04-AP3403_LED_test J3
 U 1 1 5C2995D6
 P 6025 4750
 F 0 "J3" H 6105 4742 50  0000 L CNN
 F 1 "Conn_01x04" H 6105 4651 50  0000 L CNN
-F 2 "" H 6025 4750 50  0001 C CNN
+F 2 "Connector_PinHeader_2.54mm:PinHeader_1x04_P2.54mm_Vertical" H 6025 4750 50  0001 C CNN
 F 3 "~" H 6025 4750 50  0001 C CNN
 	1    6025 4750
@@
 $EndComp
 $Comp
-L AP3403_LED_test:Conn_01x02 J1
+L Ap3403_LED_test-rescue:Conn_01x02-AP3403_LED_test J1
 U 1 1 5C299683
 P 4000 3525
 F 0 "J1" H 3920 3200 50  0000 C CNN
 F 1 "Batt conn" H 3920 3291 50  0000 C CNN
-F 2 "" H 4000 3525 50  0001 C CNN
+F 2 "Ap3403_LED_test_fp:Molex_KK-6410-02_02x2.54mm_Straight" H 4000 3525 50  0001 C CNN
 F 3 "~" H 4000 3525 50  0001 C CNN
 	1    4000 3525
@@
 $EndComp
 $Comp
-L AP3403_LED_test:GND #PWR02
+L Ap3403_LED_test-rescue:GND-AP3403_LED_test #PWR02
 U 1 1 5C29998F
 P 4475 3875
@@
 $EndComp
 $Comp
-L AP3403_LED_test:GND #PWR01
+L Ap3403_LED_test-rescue:GND-AP3403_LED_test #PWR01
 U 1 1 5C2999A8
 P 4275 3875
@@
 VIN
 $Comp
-L AP3403_LED_test:L L1
+L Ap3403_LED_test-rescue:L-AP3403_LED_test L1
 U 1 1 5C29A048
 P 6125 3425
 F 0 "L1" V 6075 3425 50  0000 C CNN
 F 1 "22u" V 6224 3425 50  0000 C CNN
-F 2 "" H 6125 3425 50  0001 C CNN
+F 2 "Inductor_SMD:L_0805_2012Metric_Pad1.15x1.40mm_HandSolder" H 6125 3425 50  0001 C CNN
 F 3 "~" H 6125 3425 50  0001 C CNN
 	1    6125 3425
@@
 	6275 3425 6925 3425
 $Comp
-L AP3403_LED_test:C C2
+L Ap3403_LED_test-rescue:C-AP3403_LED_test C2
 U 1 1 5C29A643
 P 7300 3600
 F 0 "C2" H 7415 3646 50  0000 L CNN
 F 1 "22p" H 7415 3555 50  0000 L CNN
-F 2 "" H 7338 3450 50  0001 C CNN
+F 2 "Ap3403_LED_test_fp:C_0603_HandSoldering" H 7338 3450 50  0001 C CNN
 F 3 "~" H 7300 3600 50  0001 C CNN
 	1    7300 3600
@@
 Connection ~ 6925 3825
 $Comp
-L AP3403_LED_test:R R3
+L Ap3403_LED_test-rescue:R-AP3403_LED_test R3
 U 1 1 5C29AE9D
 P 6925 4150
 F 0 "R3" H 6995 4196 50  0000 L CNN
 F 1 "470k" H 6995 4105 50  0000 L CNN
-F 2 "" V 6855 4150 50  0001 C CNN
+F 2 "Ap3403_LED_test_fp:R_0603_HandSoldering" V 6855 4150 50  0001 C CNN
 F 3 "~" H 6925 4150 50  0001 C CNN
 	1    6925 4150
@@
 	6925 4300 6925 4850
 $Comp
-L AP3403_LED_test:GND #PWR06
+L Ap3403_LED_test-rescue:GND-AP3403_LED_test #PWR06
 U 1 1 5C29B4B1
 P 6925 4850
@@
 	8475 3950 8475 4000
 $Comp
-L AP3403_LED_test:R R5
+L Ap3403_LED_test-rescue:R-AP3403_LED_test R5
 U 1 1 5C29C39A
 P 7675 4150
 F 0 "R5" H 7745 4196 50  0000 L CNN
 F 1 "1.5M" H 7745 4105 50  0000 L CNN
-F 2 "" V 7605 4150 50  0001 C CNN
+F 2 "Ap3403_LED_test_fp:R_0603_HandSoldering" V 7605 4150 50  0001 C CNN
 F 3 "~" H 7675 4150 50  0001 C CNN
 	1    7675 4150
@@
 $EndComp
 $Comp
-L AP3403_LED_test:C C3
+L Ap3403_LED_test-rescue:C-AP3403_LED_test C3
 U 1 1 5C29C78E
 P 10250 3800
 F 0 "C3" H 10365 3846 50  0000 L CNN
 F 1 "10u" H 10365 3755 50  0000 L CNN
-F 2 "" H 10288 3650 50  0001 C CNN
+F 2 "Ap3403_LED_test_fp:C_0805_HandSoldering" H 10288 3650 50  0001 C CNN
 F 3 "~" H 10250 3800 50  0001 C CNN
 	1    10250 3800
@@
 	9725 3425 9725 3600
 $Comp
-L AP3403_LED_test:GND #PWR013
+L Ap3403_LED_test-rescue:GND-AP3403_LED_test #PWR013
 U 1 1 5C29CE5B
 P 10250 4025
@@
 $EndComp
 $Comp
-L AP3403_LED_test:R R7
+L Ap3403_LED_test-rescue:R-AP3403_LED_test R7
 U 1 1 5C29D6DF
 P 8475 4150
 F 0 "R7" H 8545 4196 50  0000 L CNN
 F 1 "1.5M" H 8545 4105 50  0000 L CNN
-F 2 "" V 8405 4150 50  0001 C CNN
+F 2 "Ap3403_LED_test_fp:R_0603_HandSoldering" V 8405 4150 50  0001 C CNN
 F 3 "~" H 8475 4150 50  0001 C CNN
 	1    8475 4150
@@
 $EndComp
 $Comp
-L AP3403_LED_test:Q_NMOS_GSD Q2
+L Ap3403_LED_test-rescue:Q_NMOS_GSD-AP3403_LED_test Q2
 U 1 1 5C29D83B
 P 8375 4575
 F 0 "Q2" H 8250 4425 50  0000 L CNN
 F 1 "SI2302" H 8125 4700 50  0000 L CNN
-F 2 "" H 8575 4675 50  0001 C CNN
+F 2 "Package_TO_SOT_SMD:SOT-23_Handsoldering" H 8575 4675 50  0001 C CNN
 F 3 "~" H 8375 4575 50  0001 C CNN
 	1    8375 4575
@@
 $EndComp
 $Comp
-L AP3403_LED_test:GND #PWR08
+L Ap3403_LED_test-rescue:GND-AP3403_LED_test #PWR08
 U 1 1 5C29D9F4
 P 7675 4850
@@
 	7675 4775 7675 4850
 $Comp
-L AP3403_LED_test:GND #PWR010
+L Ap3403_LED_test-rescue:GND-AP3403_LED_test #PWR010
 U 1 1 5C29DE0D
 P 8475 4850
@@
 REG_EN
 $Comp
-L AP3403_LED_test:Q_NMOS_GSD Q3
+L Ap3403_LED_test-rescue:Q_NMOS_GSD-AP3403_LED_test Q3
 U 1 1 5C2A346A
 P 9625 4575
 F 0 "Q3" H 9500 4425 50  0000 L CNN
 F 1 "SI2302" H 9375 4700 50  0000 L CNN
-F 2 "" H 9825 4675 50  0001 C CNN
+F 2 "Package_TO_SOT_SMD:SOT-23_Handsoldering" H 9825 4675 50  0001 C CNN
 F 3 "~" H 9625 4575 50  0001 C CNN
 	1    9625 4575
@@
 	9725 3900 9725 4375
 $Comp
-L AP3403_LED_test:GND #PWR012
+L Ap3403_LED_test-rescue:GND-AP3403_LED_test #PWR012
 U 1 1 5C2A3DF1
 P 9725 4850
@@
 VLED
 $Comp
-L AP3403_LED_test:Conn_01x02 J2
+L Ap3403_LED_test-rescue:Conn_01x02-AP3403_LED_test J2
 U 1 1 5C2A850E
 P 4325 4775
 F 0 "J2" H 4245 4450 50  0000 C CNN
 F 1 "Conn_01x02" H 4245 4541 50  0000 C CNN
-F 2 "" H 4325 4775 50  0001 C CNN
+F 2 "Connector_PinHeader_2.54mm:PinHeader_1x02_P2.54mm_Vertical" H 4325 4775 50  0001 C CNN
 F 3 "~" H 4325 4775 50  0001 C CNN
 	1    4325 4775
@@
 Connection ~ 4675 4775
 $Comp
-L AP3403_LED_test:GND #PWR03
+L Ap3403_LED_test-rescue:GND-AP3403_LED_test #PWR03
 U 1 1 5C2A9919
 P 4675 4900
@@
 $EndComp
 $Comp
-L AP3403_LED_test:R R1
+L Ap3403_LED_test-rescue:R-AP3403_LED_test R1
 U 1 1 5C2AC35B
 P 4825 4100
 F 0 "R1" H 4895 4146 50  0000 L CNN
 F 1 "470k" H 4895 4055 50  0000 L CNN
-F 2 "" V 4755 4100 50  0001 C CNN
+F 2 "Ap3403_LED_test_fp:R_0603_HandSoldering" V 4755 4100 50  0001 C CNN
 F 3 "~" H 4825 4100 50  0001 C CNN
 	1    4825 4100
@@
 $EndComp
 $Comp
-L AP3403_LED_test:GND #PWR04
+L Ap3403_LED_test-rescue:GND-AP3403_LED_test #PWR04
 U 1 1 5C2ACEF4
 P 4825 4275
@@
 	4825 3925 5175 3925
 $Comp
-L AP3403_LED_test:R R4
+L Ap3403_LED_test-rescue:R-AP3403_LED_test R4
 U 1 1 5C2A0A0F
 P 7150 5075
 F 0 "R4" H 7220 5121 50  0000 L CNN
 F 1 "470k" H 7220 5030 50  0000 L CNN
-F 2 "" V 7080 5075 50  0001 C CNN
+F 2 "Ap3403_LED_test_fp:R_0603_HandSoldering" V 7080 5075 50  0001 C CNN
 F 3 "~" H 7150 5075 50  0001 C CNN
 	1    7150 5075
@@
 	7150 5225 7150 5275
 $Comp
-L AP3403_LED_test:GND #PWR07
+L Ap3403_LED_test-rescue:GND-AP3403_LED_test #PWR07
 U 1 1 5C2A22CE
 P 7150 5275
@@
 $EndComp
 $Comp
-L AP3403_LED_test:R R6
+L Ap3403_LED_test-rescue:R-AP3403_LED_test R6
 U 1 1 5C2A23C3
 P 7925 5075
 F 0 "R6" H 7995 5121 50  0000 L CNN
 F 1 "470k" H 7995 5030 50  0000 L CNN
-F 2 "" V 7855 5075 50  0001 C CNN
+F 2 "Ap3403_LED_test_fp:R_0603_HandSoldering" V 7855 5075 50  0001 C CNN
 F 3 "~" H 7925 5075 50  0001 C CNN
 	1    7925 5075
@@
 	7925 4575 8175 4575
 $Comp
-L AP3403_LED_test:GND #PWR09
+L Ap3403_LED_test-rescue:GND-AP3403_LED_test #PWR09
 U 1 1 5C2A4A37
 P 7925 5275
@@
 	7925 5225 7925 5275
 $Comp
-L AP3403_LED_test:R R8
+L Ap3403_LED_test-rescue:R-AP3403_LED_test R8
 U 1 1 5C2A852B
 P 9125 5075
 F 0 "R8" H 9195 5121 50  0000 L CNN
 F 1 "470k" H 9195 5030 50  0000 L CNN
-F 2 "" V 9055 5075 50  0001 C CNN
+F 2 "Ap3403_LED_test_fp:R_0603_HandSoldering" V 9055 5075 50  0001 C CNN
 F 3 "~" H 9125 5075 50  0001 C CNN
 	1    9125 5075
@@
 	9125 4575 9425 4575
 $Comp
-L AP3403_LED_test:GND #PWR011
+L Ap3403_LED_test-rescue:GND-AP3403_LED_test #PWR011
 U 1 1 5C2A944B
 P 9125 5275
@@
 	7150 4575 7375 4575
 $Comp
-L AP3403_LED_test:Test_Point TP1
+L Ap3403_LED_test-rescue:Test_Point-AP3403_LED_test TP1
 U 1 1 5C2BAE84
 P 6500 3750
 F 0 "TP1" H 6558 3870 50  0000 L CNN
 F 1 "FB_TP" H 6558 3779 50  0000 L CNN
-F 2 "" H 6700 3750 50  0001 C CNN
+F 2 "Ap3403_LED_test_fp:Measurement_Point_Round-SMD-Pad_Small" H 6700 3750 50  0001 C CNN
 F 3 "~" H 6700 3750 50  0001 C CNN
 	1    6500 3750
