File: senseBe_rev2/senseBe_Tx.sch (KiCad schematic (older format))
At the start: 18 parts, among them Q5 SI2302, Q6 SI2302, Q7 SI2302, U3 AP3403

Commit message: Adds PCB Design and Gerber files.
Parts:
- removed Q5, Q6, Q7: SI2302, senseBe_rev2_fp:SOT-23_Handsoldering, symbol senseBe_rev1-rescue:Q_NMOS_GSD-AP3403_LED_test-Ap3403_LED_test-rescue-senseBeTx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
- added Q3, Q4: Q_DUAL_NMOS_DMN2990UDJ-7, senseBe_rev2_fp:DMN2990UDJ-7, symbol q_dual_nmos_g1s2g2d2s1d1:Q_DUAL_NMOS_DMN2990UDJ-7
Connections:
- net GND: now also Q3.4 (S), Q4.1 (S), Q4.4 (S)
- net IR_LED_EN: now also Q3.5 (G)
- net PWR1: now also Q4.2 (G)
- net PWR2: now also Q4.5 (G)
- net at R13.2: now also Q4.6 (D)
- net at D3.1 (K): now also Q3.3 (D)
- net at R15.2: now also Q4.3 (D)
Changed lines of the file:
@@
-$EndComp
-$Comp
-L senseBe_rev1-rescue:Q_NMOS_GSD-AP3403_LED_test-Ap3403_LED_test-rescue-senseBeTx_rev3-rescue-senseBe_rev1-rescue Q?
-U 1 1 5C8021BF
-P 8050 4550
-AR Path="/5C8021BF" Ref="Q?"  Part="1"
-AR Path="/5C63BFE8/5C8021BF" Ref="Q6"  Part="1"
-F 0 "Q6" H 7950 4400 50  0000 L CNN
-F 1 "SI2302" H 7775 4675 50  0000 L CNN
-F 2 "senseBe_rev2_fp:SOT-23_Handsoldering" H 8250 4650 50  0001 C CNN
-F 3 "~" H 8050 4550 50  0001 C CNN
-	1    8050 4550
-	1    0    0    -1
 $EndComp
 $Comp
@@
 $EndComp
 $Comp
-L senseBe_rev1-rescue:Q_NMOS_GSD-AP3403_LED_test-Ap3403_LED_test-rescue-senseBeTx_rev3-rescue-senseBe_rev1-rescue Q?
-U 1 1 5C80221D
-P 9225 4550
-AR Path="/5C80221D" Ref="Q?"  Part="1"
-AR Path="/5C63BFE8/5C80221D" Ref="Q7"  Part="1"
-F 0 "Q7" H 9100 4400 50  0000 L CNN
-F 1 "SI2302" H 8975 4675 50  0000 L CNN
-F 2 "senseBe_rev2_fp:SOT-23_Handsoldering" H 9425 4650 50  0001 C CNN
-F 3 "~" H 9225 4550 50  0001 C CNN
-	1    9225 4550
-	1    0    0    -1
-$EndComp
-$Comp
 L senseBe_rev1-rescue:GND-AP3403_LED_test-Ap3403_LED_test-rescue-senseBeTx_rev3-rescue-senseBe_rev1-rescue #PWR?
 U 1 1 5C802224
@@
 Wire Wire Line
 	8150 4275 8150 4350
-$Comp
-L senseBe_rev1-rescue:Q_NMOS_GSD-AP3403_LED_test-Ap3403_LED_test-rescue-senseBeTx_rev3-rescue-senseBe_rev1-rescue Q?
-U 1 1 5C802235
-P 2650 2825
-AR Path="/5C802235" Ref="Q?"  Part="1"
-AR Path="/5C63BFE8/5C802235" Ref="Q5"  Part="1"
-F 0 "Q5" H 2525 2675 50  0000 L CNN
-F 1 "SI2302" H 2400 2950 50  0000 L CNN
-F 2 "senseBe_rev2_fp:SOT-23_Handsoldering" H 2850 2925 50  0001 C CNN
-F 3 "~" H 2650 2825 50  0001 C CNN
-	1    2650 2825
-	1    0    0    -1
-$EndComp
 $Comp
 L senseBe_rev1-rescue:GND-AP3403_LED_test-Ap3403_LED_test-rescue-senseBeTx_rev3-rescue-senseBe_rev1-rescue #PWR?
@@
 Wire Wire Line
 	9325 4250 9325 4350
+$Comp
+L q_dual_nmos_g1s2g2d2s1d1:Q_DUAL_NMOS_DMN2990UDJ-7 Q?
+U 2 1 5C6E9E9B
+P 2650 2825
+AR Path="/5C6E9E9B" Ref="Q?"  Part="2"
+AR Path="/5C63BFE8/5C6E9E9B" Ref="Q3"  Part="2"
+F 0 "Q3" H 2475 2725 50  0000 L CNN
+F 1 "Q_DUAL_NMOS_DMN2990UDJ-7" H 1700 3125 50  0000 L CNN
+F 2 "senseBe_rev2_fp:DMN2990UDJ-7" H 2850 2825 50  0001 C CNN
+F 3 "~" H 2850 2825 50  0001 C CNN
+	2    2650 2825
+	1    0    0    -1
+$EndComp
+$Comp
+L q_dual_nmos_g1s2g2d2s1d1:Q_DUAL_NMOS_DMN2990UDJ-7 Q?
+U 2 1 5C6EB2FB
+P 9225 4550
+AR Path="/5C6EB2FB" Ref="Q?"  Part="2"
+AR Path="/5C63BFE8/5C6EB2FB" Ref="Q4"  Part="2"
+F 0 "Q4" H 9050 4450 50  0000 L CNN
+F 1 "Q_DUAL_NMOS_DMN2990UDJ-7" H 8900 5100 50  0000 L CNN
+F 2 "senseBe_rev2_fp:DMN2990UDJ-7" H 9425 4550 50  0001 C CNN
+F 3 "~" H 9425 4550 50  0001 C CNN
+	2    9225 4550
+	1    0    0    -1
+$EndComp
+$Comp
+L q_dual_nmos_g1s2g2d2s1d1:Q_DUAL_NMOS_DMN2990UDJ-7 Q?
+U 1 1 5C6F3100
+P 8050 4550
+AR Path="/5C6F3100" Ref="Q?"  Part="1"
+AR Path="/5C63BFE8/5C6F3100" Ref="Q4"  Part="1"
+F 0 "Q4" H 7850 4650 50  0000 L CNN
+F 1 "Q_DUAL_NMOS_DMN2990UDJ-7" H 7650 3900 50  0000 L CNN
+F 2 "senseBe_rev2_fp:DMN2990UDJ-7" H 8250 4550 50  0001 C CNN
+F 3 "~" H 8250 4550 50  0001 C CNN
+	1    8050 4550
+	1    0    0    -1
+$EndComp
 $EndSCHEMATC

Commit message: senseBe_rev2 PCB and Gerber files modified.
Parts:
- L3: footprint Inductor_THT:L_Radial_D12.0mm_P5.00mm_Fastron_11P -> senseBe_rev2_fp:L_Radial_D12.0mm_P5.00mm_Fastron_11P
Changed lines of the file:
@@
 F 0 "L3" V 7375 2575 50  0000 C CNN
 F 1 "22u" V 7524 2575 50  0000 C CNN
-F 2 "Inductor_THT:L_Radial_D12.0mm_P5.00mm_Fastron_11P" H 7425 2575 50  0001 C CNN
+F 2 "senseBe_rev2_fp:L_Radial_D12.0mm_P5.00mm_Fastron_11P" H 7425 2575 50  0001 C CNN
 F 3 "~" H 7425 2575 50  0001 C CNN
 	1    7425 2575

Commit message: Minor changes of fixing the power Molex connector and traces to Dual MOSFET's SOT963 package.
Parts:
- C10, C11, C9: symbol senseBe_rev1-rescue:C-AP3403_LED_test-Ap3403_LED_test-rescue-senseBeTx_rev3-rescue-senseBe_rev1-rescue -> senseBe_rev2-rescue:C-AP3403_LED_test-Ap3403_LED_test-rescue-senseBeTx_rev3-rescue-senseBe_rev1-rescue-senseBe_rev1-res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
- D3: symbol senseBe_rev1-rescue:LED-AP3403_LED_test-Ap3403_LED_test-rescue-senseBeTx_rev3-rescue-senseBe_rev1-rescue -> senseBe_rev2-rescue:LED-AP3403_LED_test-Ap3403_LED_test-rescue-senseBeTx_rev3-rescue-senseBe_rev1-rescue-senseBe_rev1-r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
- L3: symbol senseBe_rev1-rescue:L-AP3403_LED_test-Ap3403_LED_test-rescue-senseBeTx_rev3-rescue-senseBe_rev1-rescue -> senseBe_rev2-rescue:L-AP3403_LED_test-Ap3403_LED_test-rescue-senseBeTx_rev3-rescue-senseBe_rev1-rescue-senseBe_rev1-res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
- Q3, Q4: symbol q_dual_nmos_g1s2g2d2s1d1:Q_DUAL_NMOS_DMN2990UDJ-7 -> senseBe_rev2-rescue:Q_DUAL_NMOS_DMN2990UDJ-7-q_dual_nmos_g1s2g2d2s1d1
- R10, R11, R12, R13, R14, R15, R8, R9: symbol senseBe_rev1-rescue:R-AP3403_LED_test-Ap3403_LED_test-rescue-senseBeTx_rev3-rescue-senseBe_rev1-rescue -> senseBe_rev2-rescue:R-AP3403_LED_test-Ap3403_LED_test-rescue-senseBeTx_rev3-rescue-senseBe_rev1-rescue-senseBe_rev1-res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
- TP1: symbol senseBe_rev1-rescue:Test_Point-AP3403_LED_test-Ap3403_LED_test-rescue-senseBeTx_rev3-rescue-senseBe_rev1-rescue -> senseBe_rev2-rescue:Test_Point-AP3403_LED_test-Ap3403_LED_test-rescue-senseBeTx_rev3-rescue-senseBe_rev1-rescue-senseBe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
- U3: symbol senseBe_rev1-rescue:AP3403-AP3403_LED_test-Ap3403_LED_test-rescue-senseBeTx_rev3-rescue-senseBe_rev1-rescue -> senseBe_rev2-rescue:AP3403-AP3403_LED_test-Ap3403_LED_test-rescue-senseBeTx_rev3-rescue-senseBe_rev1-rescue-senseBe_rev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
Changed lines of the file:
@@
 Infra Red LED Tx
 $Comp
-L senseBe_rev1-rescue:AP3403-AP3403_LED_test-Ap3403_LED_test-rescue-senseBeTx_rev3-rescue-senseBe_rev1-rescue U?
+L senseBe_rev2-rescue:AP3403-AP3403_LED_test-Ap3403_LED_test-rescue-senseBeTx_rev3-rescue-senseBe_rev1-rescue-senseBe_rev1-rescue U?
 U 1 1 5C8021A4
 P 6825 2825
@@
 $EndComp
 $Comp
-L senseBe_rev1-rescue:R-AP3403_LED_test-Ap3403_LED_test-rescue-senseBeTx_rev3-rescue-senseBe_rev1-rescue R?
+L senseBe_rev2-rescue:R-AP3403_LED_test-Ap3403_LED_test-rescue-senseBeTx_rev3-rescue-senseBe_rev1-rescue-senseBe_rev1-rescue R?
 U 1 1 5C8021AB
 P 8225 2750
@@
 $EndComp
 $Comp
-L senseBe_rev1-rescue:C-AP3403_LED_test-Ap3403_LED_test-rescue-senseBeTx_rev3-rescue-senseBe_rev1-rescue C?
+L senseBe_rev2-rescue:C-AP3403_LED_test-Ap3403_LED_test-rescue-senseBeTx_rev3-rescue-senseBe_rev1-rescue-senseBe_rev1-rescue C?
 U 1 1 5C8021B2
 P 5550 2850
@@
 $EndComp
 $Comp
-L senseBe_rev1-rescue:GND-AP3403_LED_test-Ap3403_LED_test-rescue-senseBeTx_rev3-rescue-senseBe_rev1-rescue #PWR?
+L senseBe_rev2-rescue:GND-AP3403_LED_test-Ap3403_LED_test-rescue-senseBeTx_rev3-rescue-senseBe_rev1-rescue-senseBe_rev1-rescue #PWR?
 U 1 1 5C8021B9
 P 7475 3150
@@
 $EndComp
 $Comp
-L senseBe_rev1-rescue:LED-AP3403_LED_test-Ap3403_LED_test-rescue-senseBeTx_rev3-rescue-senseBe_rev1-rescue D?
+L senseBe_rev2-rescue:LED-AP3403_LED_test-Ap3403_LED_test-rescue-senseBeTx_rev3-rescue-senseBe_rev1-rescue-senseBe_rev1-rescue D?
 U 1 1 5C8021C6
 P 3250 2575
@@
 $EndComp
 $Comp
-L senseBe_rev1-rescue:GND-AP3403_LED_test-Ap3403_LED_test-rescue-senseBeTx_rev3-rescue-senseBe_rev1-rescue #PWR?
+L senseBe_rev2-rescue:GND-AP3403_LED_test-Ap3403_LED_test-rescue-senseBeTx_rev3-rescue-senseBe_rev1-rescue-senseBe_rev1-rescue #PWR?
 U 1 1 5C8021CD
 P 5550 3400
@@
 	7175 2975 7475 2975
 $Comp
-L senseBe_rev1-rescue:L-AP3403_LED_test-Ap3403_LED_test-rescue-senseBeTx_rev3-rescue-senseBe_rev1-rescue L?
+L senseBe_rev2-rescue:L-AP3403_LED_test-Ap3403_LED_test-rescue-senseBeTx_rev3-rescue-senseBe_rev1-rescue-senseBe_rev1-rescue L?
 U 1 1 5C8021D8
 P 7425 2575
@@
 	7575 2575 8225 2575
 $Comp
-L senseBe_rev1-rescue:C-AP3403_LED_test-Ap3403_LED_test-rescue-senseBeTx_rev3-rescue-senseBe_rev1-rescue C?
+L senseBe_rev2-rescue:C-AP3403_LED_test-Ap3403_LED_test-rescue-senseBeTx_rev3-rescue-senseBe_rev1-rescue-senseBe_rev1-rescue C?
 U 1 1 5C8021E2
 P 8600 2750
@@
 Connection ~ 8225 2975
 $Comp
-L senseBe_rev1-rescue:R-AP3403_LED_test-Ap3403_LED_test-rescue-senseBeTx_rev3-rescue-senseBe_rev1-rescue R?
+L senseBe_rev2-rescue:R-AP3403_LED_test-Ap3403_LED_test-rescue-senseBeTx_rev3-rescue-senseBe_rev1-rescue-senseBe_rev1-rescue R?
 U 1 1 5C8021F4
 P 8225 3425
@@
 	8225 3575 8225 3750
 $Comp
-L senseBe_rev1-rescue:GND-AP3403_LED_test-Ap3403_LED_test-rescue-senseBeTx_rev3-rescue-senseBe_rev1-rescue #PWR?
+L senseBe_rev2-rescue:GND-AP3403_LED_test-Ap3403_LED_test-rescue-senseBeTx_rev3-rescue-senseBe_rev1-rescue-senseBe_rev1-rescue #PWR?
 U 1 1 5C8021FC
 P 8225 3750
@@
 $EndComp
 $Comp
-L senseBe_rev1-rescue:R-AP3403_LED_test-Ap3403_LED_test-rescue-senseBeTx_rev3-rescue-senseBe_rev1-rescue R?
+L senseBe_rev2-rescue:R-AP3403_LED_test-Ap3403_LED_test-rescue-senseBeTx_rev3-rescue-senseBe_rev1-rescue-senseBe_rev1-rescue R?
 U 1 1 5C802202
 P 8600 3425
@@
 $EndComp
 $Comp
-L senseBe_rev1-rescue:C-AP3403_LED_test-Ap3403_LED_test-rescue-senseBeTx_rev3-rescue-senseBe_rev1-rescue C?
+L senseBe_rev2-rescue:C-AP3403_LED_test-Ap3403_LED_test-rescue-senseBeTx_rev3-rescue-senseBe_rev1-rescue-senseBe_rev1-rescue C?
 U 1 1 5C802209
 P 3725 3025
@@
 $EndComp
 $Comp
-L senseBe_rev1-rescue:GND-AP3403_LED_test-Ap3403_LED_test-rescue-senseBeTx_rev3-rescue-senseBe_rev1-rescue #PWR?
+L senseBe_rev2-rescue:GND-AP3403_LED_test-Ap3403_LED_test-rescue-senseBeTx_rev3-rescue-senseBe_rev1-rescue-senseBe_rev1-rescue #PWR?
 U 1 1 5C802210
 P 3725 3350
@@
 $EndComp
 $Comp
-L senseBe_rev1-rescue:R-AP3403_LED_test-Ap3403_LED_test-rescue-senseBeTx_rev3-rescue-senseBe_rev1-rescue R?
+L senseBe_rev2-rescue:R-AP3403_LED_test-Ap3403_LED_test-rescue-senseBeTx_rev3-rescue-senseBe_rev1-rescue-senseBe_rev1-rescue R?
 U 1 1 5C802216
 P 8950 3425
@@
 $EndComp
 $Comp
-L senseBe_rev1-rescue:GND-AP3403_LED_test-Ap3403_LED_test-rescue-senseBeTx_rev3-rescue-senseBe_rev1-rescue #PWR?
+L senseBe_rev2-rescue:GND-AP3403_LED_test-Ap3403_LED_test-rescue-senseBeTx_rev3-rescue-senseBe_rev1-rescue-senseBe_rev1-rescue #PWR?
 U 1 1 5C802224
 P 8150 4825
@@
 	8150 4750 8150 4825
 $Comp
-L senseBe_rev1-rescue:GND-AP3403_LED_test-Ap3403_LED_test-rescue-senseBeTx_rev3-rescue-senseBe_rev1-rescue #PWR?
+L senseBe_rev2-rescue:GND-AP3403_LED_test-Ap3403_LED_test-rescue-senseBeTx_rev3-rescue-senseBe_rev1-rescue-senseBe_rev1-rescue #PWR?
 U 1 1 5C80222B
 P 9325 4825
@@
 	8150 4275 8150 4350
 $Comp
-L senseBe_rev1-rescue:GND-AP3403_LED_test-Ap3403_LED_test-rescue-senseBeTx_rev3-rescue-senseBe_rev1-rescue #PWR?
+L senseBe_rev2-rescue:GND-AP3403_LED_test-Ap3403_LED_test-rescue-senseBeTx_rev3-rescue-senseBe_rev1-rescue-senseBe_rev1-rescue #PWR?
 U 1 1 5C80223C
 P 2750 3350
@@
 VLED
 $Comp
-L senseBe_rev1-rescue:R-AP3403_LED_test-Ap3403_LED_test-rescue-senseBeTx_rev3-rescue-senseBe_rev1-rescue R?
+L senseBe_rev2-rescue:R-AP3403_LED_test-Ap3403_LED_test-rescue-senseBeTx_rev3-rescue-senseBe_rev1-rescue-senseBe_rev1-rescue R?
 U 1 1 5C802247
 P 6125 3250
@@
 $EndComp
 $Comp
-L senseBe_rev1-rescue:GND-AP3403_LED_test-Ap3403_LED_test-rescue-senseBeTx_rev3-rescue-senseBe_rev1-rescue #PWR?
+L senseBe_rev2-rescue:GND-AP3403_LED_test-Ap3403_LED_test-rescue-senseBeTx_rev3-rescue-senseBe_rev1-rescue-senseBe_rev1-rescue #PWR?
 U 1 1 5C80224E
 P 6125 3425
@@
 	6125 3075 6475 3075
 $Comp
-L senseBe_rev1-rescue:R-AP3403_LED_test-Ap3403_LED_test-rescue-senseBeTx_rev3-rescue-senseBe_rev1-rescue R?
+L senseBe_rev2-rescue:R-AP3403_LED_test-Ap3403_LED_test-rescue-senseBeTx_rev3-rescue-senseBe_rev1-rescue-senseBe_rev1-rescue R?
 U 1 1 5C802257
 P 7625 5050
@@
 	7625 5200 7625 5250
 $Comp
-L senseBe_rev1-rescue:GND-AP3403_LED_test-Ap3403_LED_test-rescue-senseBeTx_rev3-rescue-senseBe_rev1-rescue #PWR?
+L senseBe_rev2-rescue:GND-AP3403_LED_test-Ap3403_LED_test-rescue-senseBeTx_rev3-rescue-senseBe_rev1-rescue-senseBe_rev1-rescue #PWR?
 U 1 1 5C802260
 P 7625 5250
@@
 $EndComp
 $Comp
-L senseBe_rev1-rescue:R-AP3403_LED_test-Ap3403_LED_test-rescue-senseBeTx_rev3-rescue-senseBe_rev1-rescue R?
+L senseBe_rev2-rescue:R-AP3403_LED_test-Ap3403_LED_test-rescue-senseBeTx_rev3-rescue-senseBe_rev1-rescue-senseBe_rev1-rescue R?
 U 1 1 5C802266
 P 8775 5050
@@
 	8775 4550 9025 4550
 $Comp
-L senseBe_rev1-rescue:GND-AP3403_LED_test-Ap3403_LED_test-rescue-senseBeTx_rev3-rescue-senseBe_rev1-rescue #PWR?
+L senseBe_rev2-rescue:GND-AP3403_LED_test-Ap3403_LED_test-rescue-senseBeTx_rev3-rescue-senseBe_rev1-rescue-senseBe_rev1-rescue #PWR?
 U 1 1 5C80226F
 P 8775 5250
@@
 $EndComp
 $Comp
-L senseBe_rev1-rescue:R-AP3403_LED_test-Ap3403_LED_test-rescue-senseBeTx_rev3-rescue-senseBe_rev1-rescue R?
+L senseBe_rev2-rescue:R-AP3403_LED_test-Ap3403_LED_test-rescue-senseBeTx_rev3-rescue-senseBe_rev1-rescue-senseBe_rev1-rescue R?
 U 1 1 5C802275
 P 2150 3125
@@
 	2150 2825 2450 2825
 $Comp
-L senseBe_rev1-rescue:GND-AP3403_LED_test-Ap3403_LED_test-rescue-senseBeTx_rev3-rescue-senseBe_rev1-rescue #PWR?
+L senseBe_rev2-rescue:GND-AP3403_LED_test-Ap3403_LED_test-rescue-senseBeTx_rev3-rescue-senseBe_rev1-rescue-senseBe_rev1-rescue #PWR?
 U 1 1 5C80227E
 P 2150 3350
@@
 	7625 4550 7850 4550
 $Comp
-L senseBe_rev1-rescue:Test_Point-AP3403_LED_test-Ap3403_LED_test-rescue-senseBeTx_rev3-rescue-senseBe_rev1-rescue TP?
+L senseBe_rev2-rescue:Test_Point-AP3403_LED_test-Ap3403_LED_test-rescue-senseBeTx_rev3-rescue-senseBe_rev1-rescue-senseBe_rev1-rescue TP?
 U 1 1 5C802286
 P 7800 2900
@@
 	7800 2975 8225 2975
 $Comp
-L senseBe_rev1-rescue:VDD-senseBeRx_rev1-senseBeTx_rev3-rescue-senseBe_rev1-rescue #PWR?
+L senseBe_rev2-rescue:VDD-senseBeRx_rev1-senseBeTx_rev3-rescue-senseBe_rev1-rescue-senseBe_rev1-rescue #PWR?
 U 1 1 5C802290
 P 5350 2575
@@
 Connection ~ 8600 2575
 $Comp
-L senseBe_rev1-rescue:LOGO-senseBeRx_rev1-senseBeRx_rev2-rescue-senseBeRx_rev3-rescue-senseBe_rev1-rescue #G?
+L senseBe_rev2-rescue:LOGO-senseBeRx_rev1-senseBeRx_rev2-rescue-senseBeRx_rev3-rescue-senseBe_rev1-rescue-senseBe_rev1-rescue #G?
 U 1 1 5C815A89
 P 10850 6850
@@
 	9325 4250 9325 4350
 $Comp
-L q_dual_nmos_g1s2g2d2s1d1:Q_DUAL_NMOS_DMN2990UDJ-7 Q?
+L senseBe_rev2-rescue:Q_DUAL_NMOS_DMN2990UDJ-7-q_dual_nmos_g1s2g2d2s1d1 Q?
 U 2 1 5C6E9E9B
 P 2650 2825
@@
 $EndComp
 $Comp
-L q_dual_nmos_g1s2g2d2s1d1:Q_DUAL_NMOS_DMN2990UDJ-7 Q?
+L senseBe_rev2-rescue:Q_DUAL_NMOS_DMN2990UDJ-7-q_dual_nmos_g1s2g2d2s1d1 Q?
 U 2 1 5C6EB2FB
 P 9225 4550
@@
 $EndComp
 $Comp
-L q_dual_nmos_g1s2g2d2s1d1:Q_DUAL_NMOS_DMN2990UDJ-7 Q?
+L senseBe_rev2-rescue:Q_DUAL_NMOS_DMN2990UDJ-7-q_dual_nmos_g1s2g2d2s1d1 Q?
 U 1 1 5C6F3100
 P 8050 4550
