File: senseBe_rev3/senseBe_rev3_daughter/senseBe_rev3_daughter.sch (KiCad schematic (older format))
At the start: 8 parts

Commit message: Gerber files generated
Ready to manufacture.
Parts:
- removed J?: PJ-32434_3-5mmAudioJack, senseBe_rev2_fp:PJ-32434-3_5mm-AudioJack, symbol senseBe_rev3_daughter-rescue:senseBe_rev1_PJ-32434_3-5mmAudioJack-senseBe_rev1-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
- removed MK? (x2): Mounting_Hole, senseBe_rev2_fp:MountingHole_3mm, symbol senseBe_rev3_daughter-rescue:Mounting_Hole-senseBeRx_rev1-senseBeRx_rev2-rescue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
- removed SW?: SW_DPST, senseBe_rev2_fp:Molex_KK-6410-02_02x2.54mm_Straight, symbol Connector_Generic:Conn_01x02
- added J1: Conn_02x05, Connector_PinHeader_2.54mm:PinHeader_2x05_P2.54mm_Vertical, symbol Connector_Generic:Conn_02x05_Odd_Even
- added J2: StereoSocket_3-5mm_SMD, senseBe_rev3_daughter_fp:Audio_Jack_3.5mm_Horizontal_SMD, symbol senseBe_rev3_daughter-rescue:StereoSocket_3-5mm_SMD-senseBe_rev3_daughter-rescu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
- added MK1, MK2: Mounting_Hole, senseBe_rev3_daughter_fp:MountingHole_3mm, symbol senseBe_rev3_daughter-rescue:Mounting_Hole-senseBeRx_rev1-senseBeRx_rev2-rescue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
- added SW1: SW_Push_Dual, senseBe_rev3_daughter_fp:RightAngle_Tactile_Push_Button, symbol senseBe_rev3_daughter-rescue:SW_Push_Dual-senseBe_rev3_daughter-rescue-senseBe_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
- added SW2: SW_Push_SPDT, senseBe_rev3_daughter_fp:SlideSwitch_1P2T_RightAngle, symbol Switch:SW_Push_SPDT
- BT1: renamed from BT?; footprint senseBe_rev2_fp:Molex_KK-6410-02_02x2.54mm_Straight -> senseBe_rev3_daughter_fp:Molex_KK-6410-02_02x2.54mm_Straight
- C1: renamed from C?; footprint senseBe_rev2_fp:C_0603_HandSoldering -> senseBe_rev3_daughter_fp:C_0603_HandSoldering
- C2: renamed from C?; footprint senseBe_rev2_fp:C_0805_HandSoldering -> senseBe_rev3_daughter_fp:C_0805_HandSoldering
- gave numbers to parts that had none: 1
Connections:
- net BUTTON: now also J1.1 (Pin_1), SW1.3, SW1.4
- net FOCUS: now also J1.4 (Pin_4), J2.5
- net GND: now also J1.10 (Pin_10), J2.2, SW1.1, SW1.2
- net TRIGGER: now also J1.6 (Pin_6), J2.3
- net VDD: now also J1.8 (Pin_8)
- net at BT1.1 (+): now also SW2.2 (B); no longer Q1.3 (D)
- new net: Q1.3 (D), SW2.3 (C)
- new net CAM_JACK: J1.2 (Pin_2), J2.4
- no-connect marks 0 -> 5
Other:
- moved on the sheet: BT1, C1, C2, Q1
