File: SenseCam_rev1/SenseCam_rev1.kicad_pcb (KiCad board)
At the start: 2 copper layers, 75 parts, among them J1 Conn_01x30, J2 Micro_SD_Card_Det_Hirose_DM3AT, J3 Micro_SD_Card_Det_Hirose_DM3AT, J4 Conn_01x02, J5 Conn_01x04, J6 Conn_01x06, J7 Flash board, Q1 SQA403EJ, Q2 NTK3043NT1G, Q3 NTK3043NT1G, SW1 SW_SPST, U1 TPS62056DGS, U2 TPS62841, U3 TPS62840, U4 TPS22917, U5 TXB0304RUT, U6 TXB0304RUT, U7 TPS22917, U8 STM32H750VB, Y1 20MHz, Y2 32768

Commit message: Final PCB for production
Parts:
- added G***: LOGO, senseBe_rev3_main_fp:OSHW1, B.Cu at (64.0, 130.9)
- added G***: Appiko_Logo_2, senseBe_rev3_main_fp:Appiko_Logo_2, B.Cu at (72.7, 185.3)
- added G***: Appiko_Logo_2, senseBe_rev3_main_fp:Appiko_Logo_2, F.Cu at (61.3, 161.8)
- added G***: Appiko_LOGO_img, senseBe_rev3_main_fp:Appiko_LOGO_img, B.Cu at (66.1, 179.6)
- added REF***: KiCad-Logo2_8mm_SilkScreen, senseBe_rev3_main_fp:KiCad-Logo2_8mm_SilkScreen, B.Cu at (90.7, 139.9)
- moved CDSLEEP 22.6 mm to (60.0, 137.0)
- moved CSLEEP 20.8 mm to (61.8, 135.2)
- moved GND 3.29 mm to (59.9, 132.1)
- moved C19 1.93 mm to (82.1, 138.8), turned to 180 degrees
- moved VCORE 1.88 mm to (61.1, 145.4)
- moved C9 1.86 mm to (65.7, 164.6), turned to 270 degrees
- moved L1 1.74 mm to (96.3, 138.6)
- moved C8 1.66 mm to (71.9, 164.5), turned to 270 degrees
- moved C3 1.56 mm to (92.4, 142.6)
- moved C26 0.88 mm to (89.8, 140.7), turned to 0 degrees
- moved C27 0.62 mm to (87.8, 140.7), turned to 0 degrees
- moved C28 0.20 mm to (91.1, 155.2)
- moved U4 0.15 mm to (82.7, 135.3)
- moved R1 0.12 mm to (63.6, 152.2)
- renumbered TP2 to 3V3_1V8, TP6 to CDSLEEP, TP7 to CSLEEP, TP8 to D2PWREN, TP5 to GND, TP4 to RX, TP9 to SCL, TP10 to SDA, TP3 to TX, TP1 to VCORE
Connections:
- U8 pad 15: Net-(U8-Pad15) -> /H7 pins/LDR_IN
- U8 pad 2: Net-(U8-Pad2) -> /CAM_PWR_EN
- U8 pad 23: Net-(U8-Pad23) -> /CAM_STANDBY
- U8 pad 25: Net-(U8-Pad25) -> /DCMI_NRST
- U8 pad 32: /H7 pins/LDR_IN -> Net-(U8-Pad32)
- U8 pad 36: Net-(U8-Pad36) -> /CAM_FLASH_PULSE
- U8 pad 42: Net-(U8-Pad42) -> /CAM_TRIGGER
- U8 pad 43: Net-(U8-Pad43) -> /CAM_FLASH
- U8 pad 62: Net-(U8-Pad62) -> /1V4CORE_EN*
- U8 pad 77: Net-(U8-Pad77) -> /SD_PWR_EN
- U8 pad 85: Net-(U8-Pad85) -> /1V8IO_EN
Routing:
- net GND: track 117.2 -> 268.6 mm, vias 34 -> 49
- net /CAM_FLASH_PULSE: track 0.00 -> 41.3 mm, vias 0 -> 2
- net /H7 pins/CDSLEEP: track 2.43 -> 28.6 mm, vias 0 -> 2
- net /SD_PWR_EN: track 1.64 -> 26.3 mm, vias 0 -> 3
- net /H7 pins/CSLEEP: track 3.02 -> 25.7 mm, vias 0 -> 2
- net /CAM_PWR_EN: track 0.00 -> 20.7 mm, vias 0 -> 3
- net /1V8IO_EN: track 4.73 -> 21.8 mm, vias 0 -> 2
- net /CAM_FLASH: track 0.00 -> 14.5 mm, vias 0 -> 2
- net /CAM_TRIGGER: track 0.00 -> 14.0 mm, vias 0 -> 2
- net /H7 pins/STM_NRF_BUTTON: track 62.0 -> 73.3 mm
- net /CAM_STANDBY: track 0.00 -> 9.05 mm, vias 0 -> 2
- net /1V4CORE_EN*: track 1.52 -> 10.3 mm, vias 0 -> 2
- net /DCMI_NRST: track 0.00 -> 8.39 mm, vias 0 -> 2
- net /H7 pins/VBAT: track 55.1 -> 62.0 mm
- net /H7 pins/LDR_IN: track 27.4 -> 20.8 mm
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Other:
- board outline added: 45 x 70 mm
- net class Power: trace_width 0.3 -> 0.25
- board text added: "1V8/3V3"
- board text added: "3V3"
- board text added: "FLASH"
- board text added: "GND"
- board text added: "LDR"
- board text added: "LP_RX"
- board text added: "LP_TX"
- board text added: "SWDCLK"
- board text added: "SWDIO"
- board text added: "SWITCH"
- board text added: "TX"
- board text added: "VIN"
- board text added: "WKUP"
