File: SenseCam_XHP70.2_rev1/SenseCam_XHP70.2_rev1.kicad_pcb (KiCad board)
At the start: 2 copper layers, 65 x 26 mm, 10 parts, among them J1 Conn_01x03, J2 Conn_01x03, P1 CA16372_HB-SQ-WWW, P2 CA16372_HB-SQ-WWW

Commit message: Add gerbers
Parts:
- added G***: Appiko_Logo_2, sense_fp:Appiko_Logo_2, B.Cu at (32.0, 23.0)
- added G***: Appiko_LOGO_img, sense_fp:Appiko_LOGO_img, B.Cu at (56.5, 23.5)
Routing:
- net /VIN: track 71.0 -> 60.0 mm
- net /LED4: track 18.1 -> 21.2 mm
- net /LED1: track 12.1 -> 14.1 mm
- net /LED3: track 14.5 -> 16.0 mm
- net /LED2: track 16.7 -> 17.8 mm
Other:
- outline, holes or cut-outs redrawn
- board text added: "Rev1"
- board text added: "XHP70.2"
